File: hardware/cnc-hmi/cnc-hmi.kicad_pcb (KiCad board)
At the start: 2 copper layers, 397.8 x 131.2 mm, 129 parts, among them SW1 CHERRY_MX_PCB, SW10 CHERRY_MX_PCB, SW11 CHERRY_MX_PCB, SW12 CHERRY_MX_PCB, SW13 CHERRY_MX_PCB, SW14 CHERRY_MX_PCB, SW15 CHERRY_MX_PCB, SW16 CHERRY_MX_PCB, SW17 CHERRY_MX_PCB, SW18 CHERRY_MX_PCB, SW19 CHERRY_MX_PCB, SW2 CHERRY_MX_PCB, SW20 CHERRY_MX_PCB, SW21 CHERRY_MX_PCB, SW22 CHERRY_MX_PCB, SW23 CHERRY_MX_PCB, SW24 CHERRY_MX_PCB, SW25 CHERRY_MX_PCB, SW26 CHERRY_MX_PCB, SW27 CHERRY_MX_PCB, SW28 CHERRY_MX_PCB, SW29 CHERRY_MX_PCB, SW3 CHERRY_MX_PCB, SW30 CHERRY_MX_PCB, SW31 CHERRY_MX_PCB, SW32 CHERRY_MX_PCB, SW33 CHERRY_MX_PCB, SW34 CHERRY_MX_PCB, SW35 CHERRY_MX_PCB, SW36 CHERRY_MX_PCB, SW37 CHERRY_MX_PCB, SW38 CHERRY_MX_PCB, SW39 CHERRY_MX_PCB, SW4 CHERRY_MX_PCB, SW40 CHERRY_MX_PCB, SW41 CHERRY_MX_PCB, SW42 CHERRY_MX_PCB, SW43 CHERRY_MX_PCB, SW44 CHERRY_MX_PCB, SW45 CHERRY_MX_PCB, SW46 CHERRY_MX_PCB, SW47 CHERRY_MX_PCB, SW48 CHERRY_MX_PCB, SW49 CHERRY_MX_PCB, SW5 CHERRY_MX_PCB, SW50 CHERRY_MX_PCB, SW6 CHERRY_MX_PCB, SW7 CHERRY_MX_PCB, SW8 CHERRY_MX_PCB, SW9 CHERRY_MX_PCB, U1 TCA8418RTWR, U2 TLC59116FIPWR

Commit message: hw wip
Parts:
- added R10: 10K, Resistor_SMD:R_0603_1608Metric, B.Cu at (215.9, 68.8)
- added R11: 10K, Resistor_SMD:R_0603_1608Metric, B.Cu at (202.6, 70.6)
- added R12: 10K, Resistor_SMD:R_0603_1608Metric, B.Cu at (202.6, 67.6)
- added R13: 10K, Resistor_SMD:R_0603_1608Metric, B.Cu at (202.6, 64.5)
- added R14: 10K, Resistor_SMD:R_0603_1608Metric, B.Cu at (309.6, 121.2)
- added R15: 10K, Resistor_SMD:R_0603_1608Metric, B.Cu at (307.6, 159.8)
- added R16: 10K, Resistor_SMD:R_0603_1608Metric, B.Cu at (309.3, 82.3)
- added R8: 10K, Resistor_SMD:R_0603_1608Metric, B.Cu at (216.0, 63.0)
- added R9: 10K, Resistor_SMD:R_0603_1608Metric, B.Cu at (215.9, 65.3)
- added S1: REC16K25-201, CNC-HMI:REC16K25201, F.Cu at (305.4, 75.2)
- added S2: REC16K25-201, CNC-HMI:REC16K25201, F.Cu at (305.4, 113.3)
- added S3: REC16K25-201, CNC-HMI:REC16K25201, F.Cu at (305.4, 151.4)
- added U3: 74LCX07, Package_SO:SOIC-14_3.9x8.7mm_P1.27mm, B.Cu at (209.2, 65.8)
- U2: moved to B.Cu
- moved ST3 182.3 mm to (252.1, 151.4)
- moved ST4 148.5 mm to (252.1, 132.4)
- moved D48 127.7 mm to (255.3, 142.0)
- moved ST5 115.3 mm to (252.1, 113.3)
- moved ST6 106.9 mm to (252.1, 94.3)
- moved D47 72.9 mm to (255.6, 122.9)
- moved U2 64.5 mm to (321.8, 60.5), turned to 180 degrees
- moved D46 51.6 mm to (255.5, 103.6)
- moved D45 31.5 mm to (255.3, 84.8)
- moved D49 24.9 mm to (245.8, 65.8)
- moved D50 12.8 mm to (264.9, 65.5)
- moved D38 9.65 mm to (85.1, 142.9), turned to 0 degrees
- moved U1 5.05 mm to (107.4, 111.0), turned to -90 degrees
- moved A1 1.40 mm to (210.2, 112.3)
- moved ENC1 0.97 mm to (367.0, 141.9)
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Connections:
- net /KEY_R0 renamed KEY_R0
- net /KEY_R1 renamed KEY_R1
- net /KEY_R2 renamed KEY_R2
- net /KEY_R3 renamed KEY_R3
- net /KEY_R4 renamed KEY_R4
- net /KEY_R5 renamed KEY_R5
- net /KEY_R6 renamed KEY_R6
- A1 pad 25: unconnected-(A1-GPIO19-Pad25) -> /KEY_INT
- D1 pad 1: /KEY_C0 -> Net-(D1-K)
- D1 pad 2: Net-(D1-A) -> KEY_C0
- D10 pad 1: /KEY_C1 -> Net-(D10-K)
- D10 pad 2: Net-(D10-A) -> KEY_C1
- D11 pad 1: /KEY_C2 -> Net-(D11-K)
- D11 pad 2: Net-(D11-A) -> KEY_C2
- D12 pad 1: /KEY_C2 -> Net-(D12-K)
- D12 pad 2: Net-(D12-A) -> KEY_C3
- D13 pad 1: /KEY_C0 -> Net-(D13-K)
- D13 pad 2: Net-(D13-A) -> KEY_C0
- D14 pad 1: /KEY_C1 -> Net-(D14-K)
- D14 pad 2: Net-(D14-A) -> KEY_C1
- D15 pad 1: /KEY_C2 -> Net-(D15-K)
- D15 pad 2: Net-(D15-A) -> KEY_C2
- D16 pad 1: /KEY_C2 -> Net-(D16-K)
- D16 pad 2: Net-(D16-A) -> KEY_C3
- D17 pad 1: /KEY_C0 -> Net-(D17-K)
- D17 pad 2: Net-(D17-A) -> KEY_C0
- D18 pad 1: /KEY_C1 -> Net-(D18-K)
- D18 pad 2: Net-(D18-A) -> KEY_C1
- D19 pad 1: /KEY_C2 -> Net-(D19-K)
- D19 pad 2: Net-(D19-A) -> KEY_C2
- D2 pad 1: /KEY_C1 -> Net-(D2-K)
- D2 pad 2: Net-(D2-A) -> KEY_C1
- D20 pad 1: /KEY_C2 -> Net-(D20-K)
- D20 pad 2: Net-(D20-A) -> KEY_C3
- D21 pad 1: /KEY_C3 -> Net-(D21-K)
- D21 pad 2: Net-(D21-A) -> KEY_C4
- D22 pad 1: /KEY_C4 -> Net-(D22-K)
- D22 pad 2: Net-(D22-A) -> KEY_C5
- D23 pad 1: /KEY_C5 -> Net-(D23-K)
- D23 pad 2: Net-(D23-A) -> KEY_C6
- D24 pad 1: /KEY_C6 -> Net-(D24-K)
- D24 pad 2: Net-(D24-A) -> KEY_C7
- D25 pad 1: /KEY_C3 -> Net-(D25-K)
- D25 pad 2: Net-(D25-A) -> KEY_C4
- D26 pad 1: /KEY_C4 -> Net-(D26-K)
- D26 pad 2: Net-(D26-A) -> KEY_C5
- D27 pad 1: /KEY_C5 -> Net-(D27-K)
- D27 pad 2: Net-(D27-A) -> KEY_C6
- D28 pad 1: /KEY_C6 -> Net-(D28-K)
- D28 pad 2: Net-(D28-A) -> KEY_C7
- D29 pad 1: /KEY_C3 -> Net-(D29-K)
- D29 pad 2: Net-(D29-A) -> KEY_C4
- D3 pad 1: /KEY_C2 -> Net-(D3-K)
- D3 pad 2: Net-(D3-A) -> KEY_C2
- D30 pad 1: /KEY_C4 -> Net-(D30-K)
- D30 pad 2: Net-(D30-A) -> KEY_C5
- D31 pad 1: /KEY_C5 -> Net-(D31-K)
- D31 pad 2: Net-(D31-A) -> KEY_C6
- D32 pad 1: /KEY_C6 -> Net-(D32-K)
- D32 pad 2: Net-(D32-A) -> KEY_C7
- D33 pad 1: /KEY_C3 -> Net-(D33-K)
- D33 pad 2: Net-(D33-A) -> KEY_C4
- D34 pad 1: /KEY_C4 -> Net-(D34-K)
- D34 pad 2: Net-(D34-A) -> KEY_C5
- D35 pad 1: /KEY_C5 -> Net-(D35-K)
- D35 pad 2: Net-(D35-A) -> KEY_C6
- D36 pad 1: /KEY_C6 -> Net-(D36-K)
- D36 pad 2: Net-(D36-A) -> KEY_C7
- D37 pad 1: /KEY_C3 -> Net-(D37-K)
- D37 pad 2: Net-(D37-A) -> KEY_C4
- D38 pad 1: /KEY_C4 -> Net-(D38-K)
- D38 pad 2: Net-(D38-A) -> KEY_C5
- D39 pad 1: /KEY_C5 -> Net-(D39-K)
- D39 pad 2: Net-(D39-A) -> KEY_C6
- D4 pad 1: /KEY_C2 -> Net-(D4-K)
- D4 pad 2: Net-(D4-A) -> KEY_C3
- D40 pad 1: /KEY_C6 -> Net-(D40-K)
- D40 pad 2: Net-(D40-A) -> KEY_C7
- D41 pad 1: /KEY_C3 -> Net-(D41-K)
- D41 pad 2: Net-(D41-A) -> KEY_C4
- D42 pad 1: /KEY_C4 -> Net-(D42-K)
- D42 pad 2: Net-(D42-A) -> KEY_C5
- D43 pad 1: /KEY_C5 -> Net-(D43-K)
- D43 pad 2: Net-(D43-A) -> KEY_C6
- D44 pad 1: /KEY_C6 -> Net-(D44-K)
- D44 pad 2: Net-(D44-A) -> KEY_C7
- D45 pad 1: /KEY_C0 -> Net-(D45-K)
- D45 pad 2: Net-(D45-A) -> KEY_C0
- D46 pad 1: /KEY_C1 -> Net-(D46-K)
- D46 pad 2: Net-(D46-A) -> KEY_C1
- D47 pad 1: /KEY_C2 -> Net-(D47-K)
- D47 pad 2: Net-(D47-A) -> KEY_C2
- D48 pad 1: /KEY_C2 -> Net-(D48-K)
- D48 pad 2: Net-(D48-A) -> KEY_C3
- D49 pad 1: /KEY_C0 -> Net-(D49-K)
- D49 pad 2: Net-(D49-A) -> KEY_C0
- D5 pad 1: /KEY_C0 -> Net-(D5-K)
- D5 pad 2: Net-(D5-A) -> KEY_C0
- D50 pad 1: /KEY_C1 -> Net-(D50-K)
- D50 pad 2: Net-(D50-A) -> KEY_C1
- D6 pad 1: /KEY_C1 -> Net-(D6-K)
- D6 pad 2: Net-(D6-A) -> KEY_C1
- D7 pad 1: /KEY_C2 -> Net-(D7-K)
- D7 pad 2: Net-(D7-A) -> KEY_C2
- D8 pad 1: /KEY_C2 -> Net-(D8-K)
- D8 pad 2: Net-(D8-A) -> KEY_C3
- D9 pad 1: /KEY_C0 -> Net-(D9-K)
- D9 pad 2: Net-(D9-A) -> KEY_C0
- SW1 pad 2: Net-(D1-A) -> Net-(D1-K)
- SW10 pad 2: Net-(D10-A) -> Net-(D10-K)
- SW11 pad 2: Net-(D11-A) -> Net-(D11-K)
- SW12 pad 2: Net-(D12-A) -> Net-(D12-K)
- SW13 pad 2: Net-(D13-A) -> Net-(D13-K)
- SW14 pad 2: Net-(D14-A) -> Net-(D14-K)
- SW15 pad 2: Net-(D15-A) -> Net-(D15-K)
- SW16 pad 2: Net-(D16-A) -> Net-(D16-K)
- SW17 pad 2: Net-(D17-A) -> Net-(D17-K)
- SW18 pad 2: Net-(D18-A) -> Net-(D18-K)
- SW19 pad 2: Net-(D19-A) -> Net-(D19-K)
- SW2 pad 2: Net-(D2-A) -> Net-(D2-K)
- SW20 pad 2: Net-(D20-A) -> Net-(D20-K)
- SW21 pad 2: Net-(D21-A) -> Net-(D21-K)
- SW22 pad 2: Net-(D22-A) -> Net-(D22-K)
- SW23 pad 2: Net-(D23-A) -> Net-(D23-K)
- SW24 pad 2: Net-(D24-A) -> Net-(D24-K)
- SW25 pad 2: Net-(D25-A) -> Net-(D25-K)
- SW26 pad 2: Net-(D26-A) -> Net-(D26-K)
- SW27 pad 2: Net-(D27-A) -> Net-(D27-K)
- SW28 pad 2: Net-(D28-A) -> Net-(D28-K)
- SW29 pad 2: Net-(D29-A) -> Net-(D29-K)
- SW3 pad 2: Net-(D3-A) -> Net-(D3-K)
- SW30 pad 2: Net-(D30-A) -> Net-(D30-K)
- SW31 pad 2: Net-(D31-A) -> Net-(D31-K)
- SW32 pad 2: Net-(D32-A) -> Net-(D32-K)
- SW33 pad 2: Net-(D33-A) -> Net-(D33-K)
- SW34 pad 2: Net-(D34-A) -> Net-(D34-K)
- SW35 pad 2: Net-(D35-A) -> Net-(D35-K)
- SW36 pad 2: Net-(D36-A) -> Net-(D36-K)
- SW37 pad 2: Net-(D37-A) -> Net-(D37-K)
- SW38 pad 2: Net-(D38-A) -> Net-(D38-K)
- SW39 pad 2: Net-(D39-A) -> Net-(D39-K)
- SW4 pad 2: Net-(D4-A) -> Net-(D4-K)
- SW40 pad 2: Net-(D40-A) -> Net-(D40-K)
- SW41 pad 2: Net-(D41-A) -> Net-(D41-K)
- SW42 pad 2: Net-(D42-A) -> Net-(D42-K)
- SW43 pad 2: Net-(D43-A) -> Net-(D43-K)
- SW44 pad 2: Net-(D44-A) -> Net-(D44-K)
- SW45 pad 2: Net-(D45-A) -> Net-(D45-K)
- SW46 pad 2: Net-(D46-A) -> Net-(D46-K)
- SW47 pad 2: Net-(D47-A) -> Net-(D47-K)
- SW48 pad 2: Net-(D48-A) -> Net-(D48-K)
- SW49 pad 2: Net-(D49-A) -> Net-(D49-K)
- SW5 pad 2: Net-(D5-A) -> Net-(D5-K)
- SW50 pad 2: Net-(D50-A) -> Net-(D50-K)
- SW6 pad 2: Net-(D6-A) -> Net-(D6-K)
- SW7 pad 2: Net-(D7-A) -> Net-(D7-K)
- SW8 pad 2: Net-(D8-A) -> Net-(D8-K)
- SW9 pad 2: Net-(D9-A) -> Net-(D9-K)
- U1 pad 1: unconnected-(U1-ROW7-Pad1) -> /ENC0_SW
- U1 pad 10: /KEY_C1 -> KEY_C1
- U1 pad 11: /KEY_C2 -> KEY_C2
- U1 pad 12: /KEY_C3 -> KEY_C3
- U1 pad 13: /KEY_C4 -> KEY_C4
- U1 pad 14: /KEY_C5 -> KEY_C5
- U1 pad 15: /KEY_C6 -> KEY_C6
- U1 pad 16: /KEY_C7 -> KEY_C7
- U1 pad 17: unconnected-(U1-COL8-Pad17) -> /ENC1_SW
- U1 pad 18: unconnected-(U1-COL9-Pad18) -> /ENC2_SW
- U1 pad 24: unconnected-(U1-~{INT}-Pad24) -> /KEY_INT
- U1 pad 9: /KEY_C0 -> KEY_C0
Routing:
- net GND: track 0.00 -> 584.7 mm, vias 0 -> 18
- net KEY_R4: track 0.00 -> 581.5 mm, vias 0 -> 5
- net KEY_C4: track 0.00 -> 544.6 mm, vias 0 -> 12
- net KEY_C7: track 0.00 -> 525.3 mm, vias 0 -> 11
- net KEY_C5: track 0.00 -> 446.3 mm, vias 0 -> 10
- net KEY_R5: track 0.00 -> 441.3 mm, vias 0 -> 3
- net +3V3: track 0.00 -> 430.2 mm, vias 0 -> 18
- net KEY_C6: track 0.00 -> 417.1 mm, vias 0 -> 9
- net +5V: track 0.00 -> 398.9 mm, vias 0 -> 3
- net KEY_C3: track 0.00 -> 372.6 mm, vias 0 -> 6
- net /ENC2_SW: track 0.00 -> 367.4 mm, vias 0 -> 4
- net /ENC1_SW: track 0.00 -> 329.1 mm, vias 0 -> 4
- net /PERIPH_RESET: track 0.00 -> 278.5 mm, vias 0 -> 6
- net /ENC0_SW: track 0.00 -> 278.4 mm, vias 0 -> 4
- net /I2C0_SDA: track 0.00 -> 274.0 mm, vias 0 -> 4
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- added copper zone on B.Cu, net GND
- added copper zone on F.Cu, net GND
Other:
- board size 397.8 x 131.2 mm -> 381 x 127 mm

Commit message: Commit before rev0 release to fab
Parts:
- added C10: 0.1uF, Capacitor_SMD:C_0603_1608Metric, B.Cu at (215.9, 70.4)
- added C11: 0.1uF, Capacitor_SMD:C_0603_1608Metric, B.Cu at (305.6, 84.6)
- added C12: 0.1uF, Capacitor_SMD:C_0603_1608Metric, B.Cu at (304.8, 121.7)
- added C13: 0.1uF, Capacitor_SMD:C_0603_1608Metric, B.Cu at (304.8, 165.4)
- added C4: 0.1uF, Capacitor_SMD:C_0603_1608Metric, B.Cu at (103.1, 114.3)
- added C5: 1uF, Capacitor_SMD:C_0805_2012Metric, B.Cu at (103.1, 116.1)
- added C6: 0.1uF, Capacitor_SMD:C_0603_1608Metric, B.Cu at (318.3, 53.6)
- added C7: 1uF, Capacitor_SMD:C_0805_2012Metric, B.Cu at (320.3, 53.3)
- added C8: 0.1uF, Capacitor_SMD:C_0603_1608Metric, B.Cu at (356.9, 57.1)
- added C9: 1uF, Capacitor_SMD:C_0805_2012Metric, B.Cu at (356.9, 55.4)
- added H1: MountingHole, CNC-HMI:M3-Mounting Hole, F.Cu at (25.4, 47.5)
- added H10: MountingHole, CNC-HMI:M3-Mounting Hole, F.Cu at (398.8, 47.5)
- added H11: MountingHole, CNC-HMI:M3-Mounting Hole, F.Cu at (398.8, 166.9)
- added H14: MountingHole, CNC-HMI:M3-Mounting Hole, F.Cu at (346.7, 125.0)
- added H15: MountingHole, CNC-HMI:M3-Mounting Hole, F.Cu at (386.1, 125.0)
- added H16: MountingHole, CNC-HMI:M2.5-Mounting Hole, F.Cu at (330.2, 53.8)
- added H17: MountingHole, CNC-HMI:M2.5-Mounting Hole, F.Cu at (388.6, 53.8)
- added H2: MountingHole, CNC-HMI:M3-Mounting Hole, F.Cu at (25.4, 166.9)
- added H3: MountingHole, CNC-HMI:M3-Mounting Hole, F.Cu at (108.0, 47.5)
- added H4: MountingHole, CNC-HMI:M3-Mounting Hole, F.Cu at (108.0, 166.9)
- added H5: MountingHole, CNC-HMI:M3-Mounting Hole, F.Cu at (210.8, 47.5)
- added H6: MountingHole, CNC-HMI:M3-Mounting Hole, F.Cu at (194.3, 166.9)
- added H7: MountingHole, CNC-HMI:M3-Mounting Hole, F.Cu at (226.1, 166.9)
- added H8: MountingHole, CNC-HMI:M3-Mounting Hole, F.Cu at (290.8, 166.9)
- added H9: MountingHole, CNC-HMI:M3-Mounting Hole, F.Cu at (290.8, 47.5)
- added J1: Conn_01x03, Connector_JST:JST_PH_S3B-PH-K_1x03_P2.00mm_Horizontal, B.Cu at (235.7, 163.2)
- added J2: Conn_01x04, Connector_JST:JST_PH_S4B-PH-K_1x04_P2.00mm_Horizontal, B.Cu at (187.6, 163.1)
- added J3: Conn_01x08, Connector_JST:JST_PH_S8B-PH-K_1x08_P2.00mm_Horizontal, B.Cu at (191.8, 70.9)
- added J4: Conn_01x05, Connector_JST:JST_PH_S5B-PH-K_1x05_P2.00mm_Horizontal, B.Cu at (309.6, 59.4)
- added LED10: LED, MX_V2_Misc:MX-LED-Reversed, F.Cu at (252.1, 113.3)
- added LED11: LED, MX_V2_Misc:MX-LED-Reversed, F.Cu at (252.1, 132.4)
- added LED12: LED, MX_V2_Misc:MX-LED-Reversed, F.Cu at (252.1, 151.4)
- added LED9: LED, MX_V2_Misc:MX-LED-Reversed, F.Cu at (252.1, 94.3)
- added LOGO1: ~, CNC-HMI:LinuxCNC Logo, B.Cu at (335.3, 161.8)
- added LOGO2: Logo_Open_Hardware_Small, Symbol:OSHW-Logo_11.4x12mm_SilkScreen, B.Cu at (279.4, 161.8)
- moved LCD1 8.08 mm to (352.6, 52.6), turned to 90 degrees
- moved R7 6.82 mm to (357.1, 53.6), turned to 180 degrees
- moved C1 6.54 mm to (356.9, 51.8), turned to 180 degrees
- moved C2 3.27 mm to (356.9, 49.8), turned to 180 degrees
- moved R11 2.29 mm to (202.6, 68.3)
- moved C3 2.24 mm to (356.9, 47.8), turned to 180 degrees
- moved R12 1.02 mm to (202.6, 66.5)
Connections:
- A1 pad 24: unconnected-(A1-GPIO18-Pad24) -> /SPARE_GPIO18
- A1 pad 31: unconnected-(A1-GPIO26_ADC0-Pad31) -> /SPARE_GPIO26
- A1 pad 32: unconnected-(A1-GPIO27_ADC1-Pad32) -> /SPARE_GPIO27
- A1 pad 34: unconnected-(A1-GPIO28_ADC2-Pad34) -> /SPARE_GPIO28
- A1 pad D1: unconnected-(A1-SWCLK-PadD1) -> Net-(A1-SWCLK)
- A1 pad D3: unconnected-(A1-SWDIO-PadD3) -> Net-(A1-SWDIO)
- LCD1 pad 10: unconnected-(LCD1-VPP-Pad10) -> +3V3
- LCD1 pad 7: unconnected-(LCD1-VDD1-Pad7) -> +3V3
- U2 pad 15: unconnected-(U2-~{OUT8}-Pad15) -> Net-(LED9-K)
- U2 pad 16: unconnected-(U2-~{OUT9}-Pad16) -> Net-(LED10-K)
- U2 pad 17: unconnected-(U2-~{OUT10}-Pad17) -> Net-(LED11-K)
- U2 pad 18: unconnected-(U2-~{OUT11}-Pad18) -> Net-(LED12-K)
- U2 pad 20: unconnected-(U2-~{OUT12}-Pad20) -> /SPARE_LED12
- U2 pad 21: unconnected-(U2-~{OUT13}-Pad21) -> /SPARE_LED13
- U2 pad 22: unconnected-(U2-~{OUT14}-Pad22) -> /SPARE_LED14
- U2 pad 23: unconnected-(U2-~{OUT15}-Pad23) -> /SPARE_LED15
Routing:
- net +3V3: track 430.2 -> 728.7 mm, vias 18 -> 21
- net /LCD_A0: track 0.00 -> 263.5 mm, vias 0 -> 4
- net /SPI0_CS0: track 0.00 -> 255.7 mm, vias 0 -> 4
- net /SPI0_SCK: track 0.00 -> 254.3 mm, vias 0 -> 4
- net /SPI0_DOUT: track 0.00 -> 251.2 mm, vias 0 -> 4
- net +5V: track 398.9 -> 564.4 mm, vias 3 -> 5
- net GND: track 584.7 -> 749.1 mm, vias 18 -> 854
- net Net-(LED12-K): track 0.00 -> 163.2 mm, vias 0 -> 2
- net Net-(LED11-K): track 0.00 -> 149.3 mm, vias 0 -> 2
- net KEY_C1: track 176.5 -> 308.1 mm, vias 7 -> 10
- net Net-(LED10-K): track 0.00 -> 120.3 mm, vias 0 -> 3
- net Net-(A1-SWCLK): track 0.00 -> 107.4 mm, vias 0 -> 1
- net Net-(LED9-K): track 0.00 -> 100.0 mm, vias 0 -> 2
- net Net-(A1-SWDIO): track 0.00 -> 99.8 mm, vias 0 -> 1
- net /SPARE_GPIO28: track 0.00 -> 85.9 mm, vias 0 -> 2
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Other:
- outline, holes or cut-outs redrawn
- board text added: "DESIGNED BY STEVE RICHARDSON"
- board text added: "PI PICO SWD SWCLK-GND-SWDIO"
- board text added: "PI PICO UART RX-TX-GND-3V3"
- board text added: "RASPBERRY PI PICO2"
- board text added: "REVISION 0 2025-MAR-10"
- board text added: "SPARE I/O"
- board text added: "SPARE LEDS"
- board text added: "TANGENTAUDIO CNC USB HMI CONTROLLER"
