File: hardware/cnc-hmi/cnc-hmi.kicad_sch (KiCad schematic)
At the start: 129 parts, among them SW1 CHERRY_MX_PCB, SW10 CHERRY_MX_PCB, SW11 CHERRY_MX_PCB, SW12 CHERRY_MX_PCB, SW13 CHERRY_MX_PCB, SW14 CHERRY_MX_PCB, SW15 CHERRY_MX_PCB, SW16 CHERRY_MX_PCB, SW17 CHERRY_MX_PCB, SW18 CHERRY_MX_PCB, SW19 CHERRY_MX_PCB, SW2 CHERRY_MX_PCB, SW20 CHERRY_MX_PCB, SW21 CHERRY_MX_PCB, SW22 CHERRY_MX_PCB, SW23 CHERRY_MX_PCB, SW24 CHERRY_MX_PCB, SW25 CHERRY_MX_PCB, SW26 CHERRY_MX_PCB, SW27 CHERRY_MX_PCB, SW28 CHERRY_MX_PCB, SW29 CHERRY_MX_PCB, SW3 CHERRY_MX_PCB, SW30 CHERRY_MX_PCB, SW31 CHERRY_MX_PCB, SW32 CHERRY_MX_PCB, SW33 CHERRY_MX_PCB, SW34 CHERRY_MX_PCB, SW35 CHERRY_MX_PCB, SW36 CHERRY_MX_PCB, SW37 CHERRY_MX_PCB, SW38 CHERRY_MX_PCB, SW39 CHERRY_MX_PCB, SW4 CHERRY_MX_PCB, SW40 CHERRY_MX_PCB, SW41 CHERRY_MX_PCB, SW42 CHERRY_MX_PCB, SW43 CHERRY_MX_PCB, SW44 CHERRY_MX_PCB, SW45 CHERRY_MX_PCB, SW46 CHERRY_MX_PCB, SW47 CHERRY_MX_PCB, SW48 CHERRY_MX_PCB, SW49 CHERRY_MX_PCB, SW5 CHERRY_MX_PCB, SW50 CHERRY_MX_PCB, SW6 CHERRY_MX_PCB, SW7 CHERRY_MX_PCB, SW8 CHERRY_MX_PCB, SW9 CHERRY_MX_PCB, U1 TCA8418RTWR, U2 TLC59116FIPWR

Commit message: hw wip
Parts:
- removed D1, D10, D11, D12, D13, D14, D15, D16, D17, D18, D19, D2, D20, D21, D22, D23, D24, D25, D26, D27, D28, D29, D3, D30, D31, D32, D33, D34, D35, D36, D37, D38, D39, D4, D40, D41, D42, D43, D44, D45, D46, D47, D48, D49, D5, D50, D6, D7, D8, D9: D_Small, Diode_SMD:D_SOD-523, symbol Device:D_Small
- removed ST1, ST2, ST3, ST4, ST5, ST6: ~, CNC-HMI:Stabilizer_Cherry_MX_2.00u, symbol CNC-HMI:Cherry_MX_Stabilizer_2u
- removed SW1, SW10, SW11, SW12, SW13, SW14, SW15, SW17, SW18, SW19, SW2, SW20, SW21, SW22, SW23, SW24, SW25, SW26, SW27, SW28, SW29, SW3, SW30, SW31, SW32, SW33, SW34, SW35, SW36, SW37, SW39, SW4, SW40, SW41, SW42, SW43, SW44, SW49, SW5, SW50, SW6, SW7, SW8, SW9: CHERRY_MX_PCB, CNC-HMI:SW_Cherry_MX_PCB_1.00u, symbol Switch:SW_SPST
- removed SW16: CHERRY_MX_PCB, CNC-HMI:SW_Cherry_MX_PCB_2.00u_90deg, symbol Switch:SW_SPST
- removed SW38, SW45, SW46, SW47, SW48: CHERRY_MX_PCB, CNC-HMI:SW_Cherry_MX_PCB_2.00u, symbol Switch:SW_SPST
- added R10, R11, R12, R13, R14, R15, R16, R8, R9: 10K, Resistor_SMD:R_0603_1608Metric, symbol Device:R_US
- added S1, S2, S3: REC16K25-201, CNC-HMI:REC16K25201, symbol REC16K25-201:REC16K25-201
- added U3: 74LCX07, Package_SO:SOIC-14_3.9x8.7mm_P1.27mm, symbol 74xx:74LCX07
Connections:
- net +3V3: now also R10.1, R11.1, R12.1, R13.1, R14.1, R15.1, R16.1, R8.1, R9.1, U3.14 (VCC)
- net +5V: now also S1.6 (POWER_＋_5_V), S2.6 (POWER_＋_5_V), S3.6 (POWER_＋_5_V)
- net ENC0_A: now also R8.2, U3.2
- net ENC0_B: now also R9.2, U3.4
- net ENC1_A: now also R10.2, U3.6
- net ENC1_B: now also R11.2, U3.8
- net ENC2_A: now also R12.2, U3.10
- net ENC2_B: now also R13.2, U3.12
- net GND: now also S1.1 (POWER_0_(V)), S1.2 (FOR_SWITCH_1), S2.1 (POWER_0_(V)), S2.2 (FOR_SWITCH_1), S3.1 (POWER_0_(V)), S3.2 (FOR_SWITCH_1), U3.7 (GND)
- net ENC0_SW: now reaches U1.1 (ROW7)
- net ENC0_SW: now also R16.2, S1.3 (FOR_SWITCH_2)
- net ENC1_SW: now reaches U1.17 (COL8)
- net ENC1_SW: now also R14.2, S2.3 (FOR_SWITCH_2)
- net ENC2_SW: now reaches U1.18 (COL9)
- net ENC2_SW: now also R15.2, S3.3 (FOR_SWITCH_2)
- new net: S3.4 (OUTPUT_“B”), U3.13
- new net: S3.5 (OUTPUT_“A”), U3.11
- new net: S2.4 (OUTPUT_“B”), U3.9
- new net: S1.4 (OUTPUT_“B”), U3.3
- new net: S2.5 (OUTPUT_“A”), U3.5
- new net: S1.5 (OUTPUT_“A”), U3.1
Other:
- added sheet Keypad (keypad.kicad_sch)
- note added: "5V->3.3V LEVEL SHIFT"
- note added: "FEED/SPEED OVERRIDE ENCODER KNOBS"
- note added: "I2C LED CONTROLLER"
- note added: "I2C MATRIX KEYPAD ENCODER"
- note added: "JOG CONTROL ENCODER"
- note added: "RASPBERRY PI PICO 2"
- note added: "SPI OLED DISPLAY"
- moved on the sheet: A1, C1, C2, C3, ENC1, LCD1, LED1, LED2, LED3, LED4, LED5, LED6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

Commit message: Commit before rev0 release to fab
Parts:
- added C10, C11, C12, C13, C4, C6, C8: 0.1uF, Capacitor_SMD:C_0603_1608Metric, symbol Device:C_Small
- added C5, C7, C9: 1uF, Capacitor_SMD:C_0805_2012Metric, symbol Device:C_Small
- added H1, H10, H11, H14, H15, H2, H3, H4, H5, H6, H7, H8, H9: MountingHole, CNC-HMI:M3-Mounting Hole, symbol Mechanical:MountingHole
- added H16, H17: MountingHole, CNC-HMI:M2.5-Mounting Hole, symbol Mechanical:MountingHole
- added J1: Conn_01x03, Connector_JST:JST_PH_S3B-PH-K_1x03_P2.00mm_Horizontal, symbol Connector_Generic:Conn_01x03
- added J2: Conn_01x04, Connector_JST:JST_PH_S4B-PH-K_1x04_P2.00mm_Horizontal, symbol Connector_Generic:Conn_01x04
- added J3: Conn_01x08, Connector_JST:JST_PH_S8B-PH-K_1x08_P2.00mm_Horizontal, symbol Connector_Generic:Conn_01x08
- added J4: Conn_01x05, Connector_JST:JST_PH_S5B-PH-K_1x05_P2.00mm_Horizontal, symbol Connector_Generic:Conn_01x05
- added LED10, LED11, LED12, LED9: LED, MX_V2_Misc:MX-LED-Reversed, symbol Device:LED
- added LOGO1: ~, CNC-HMI:LinuxCNC Logo, symbol CNC-HMI:LinuxCNC_Logo
- added LOGO2: Logo_Open_Hardware_Small, Symbol:OSHW-Logo_11.4x12mm_SilkScreen, symbol Graphic:Logo_Open_Hardware_Small
Connections:
- net +3V3: now also LCD1.10 (VPP), LCD1.7 (VDD1), C10.1, C4.1, C5.1, C6.1, C7.1, C8.1, C9.1, J2.4 (Pin_4), J3.8 (Pin_8)
- net +5V: now also C11.1, C12.1, C13.1, J4.5 (Pin_5), LED10.2 (A), LED11.2 (A), LED12.2 (A), LED9.2 (A)
- net GND: now also C10.2, C11.2, C12.2, C13.2, C4.2, C5.2, C6.2, C7.2, C8.2, C9.2, J1.2 (Pin_2), J2.3 (Pin_3), J3.7 (Pin_7)
- net I2C0_SCL: now also J3.6 (Pin_6)
- net I2C0_SDA: now also J3.5 (Pin_5)
- net UART0_RX: now also J2.1 (Pin_1)
- net UART0_TX: now also J2.2 (Pin_2)
- net at U2.15 (~{OUT8}): now also LED9.1 (K)
- net at U2.16 (~{OUT9}): now also LED10.1 (K)
- net at U2.17 (~{OUT10}): now also LED11.1 (K)
- net at U2.18 (~{OUT11}): now also LED12.1 (K)
- net SPARE_LED12: now reaches U2.20 (~{OUT12})
- net SPARE_LED12: now also J4.1 (Pin_1)
- net SPARE_LED13: now reaches U2.21 (~{OUT13})
- net SPARE_LED13: now also J4.2 (Pin_2)
- net SPARE_LED14: now reaches U2.22 (~{OUT14})
- net SPARE_LED14: now also J4.3 (Pin_3)
- net SPARE_LED15: now reaches U2.23 (~{OUT15})
- net SPARE_LED15: now also J4.4 (Pin_4)
- net SPARE_GPIO18: now reaches A1.24 (GPIO18)
- net SPARE_GPIO18: now also J3.1 (Pin_1)
- net SPARE_GPIO26: now reaches A1.31 (GPIO26_ADC0)
- net SPARE_GPIO26: now also J3.2 (Pin_2)
- net SPARE_GPIO27: now reaches A1.32 (GPIO27_ADC1)
- net SPARE_GPIO27: now also J3.3 (Pin_3)
- net SPARE_GPIO28: now reaches A1.34 (GPIO28_ADC2)
- net SPARE_GPIO28: now also J3.4 (Pin_4)
- net at A1.D1 (SWCLK): now also J1.1 (Pin_1)
- net at A1.D3 (SWDIO): now also J1.3 (Pin_3)
- no-connect marks 4 -> 5
Other:
- moved on the sheet: C1, C2, C3, LCD1, LED1, LED2, LED3, LED4, LED5, LED6, LED7, LED8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
