File: hardware/cnc-hmi-encleds/cnc-hmi-encleds.kicad_pcb (KiCad board)
At the start: 2 copper layers, 32 x 108.2 mm, 48 parts, among them J1 Conn_01x04, U1 SN74LVC1T45DBV

Commit message: prep for fab&assembly
Parts:
- added C1: 0.1uF, Capacitor_SMD:C_0603_1608Metric, F.Cu at (152.3, 78.4)
- added C2: 0.1uF, Capacitor_SMD:C_0603_1608Metric, F.Cu at (150.0, 76.1)
- added C3: 1uF, Capacitor_SMD:C_0805_2012Metric, F.Cu at (152.5, 75.7)
Routing:
- net +5V: track 8.65 -> 14.0 mm
- net GND: track 54.1 -> 58.1 mm, vias 46 -> 49
- net +3V3: track 9.31 -> 11.2 mm
